File: SimpleSensoredBldcController.kicad_pcb (KiCad board)
At the start: 2 copper layers, 30 parts, among them J1 Conn_01x02_Male, Q1 80V 80A, Q2 80V 80A, Q3 80V 80A, Q4 80V 80A, Q5 80V 80A, Q6 80V 80A, U1 A4915_LP, U2 MP2565DN-LF-Z

Commit message: Started routing.
Parts:
- added C10: 470uF 63V, Capacitor_THT:C_Radial_D12.5mm_H25.0mm_P5.00mm, F.Cu at (113.1, 76.4)
- added C11: 100nF 6.3V, Capacitor_SMD:C_0603_1608Metric, F.Cu at (167.9, 76.5)
- added C12: 470uF 63V, Capacitor_THT:C_Radial_D12.5mm_H25.0mm_P5.00mm, F.Cu at (98.6, 90.5)
- added C13: 100nF 6.3V, Capacitor_SMD:C_0603_1608Metric, F.Cu at (131.9, 111.7)
- added C14: 470uF 63V, Capacitor_THT:C_Radial_D12.5mm_H25.0mm_P5.00mm, F.Cu at (98.6, 104.5)
- added C15: 220nF 16V, Capacitor_SMD:C_0603_1608Metric, F.Cu at (104.9, 130.4)
- added C16: 100nF 100V, Capacitor_SMD:C_0805_2012Metric, F.Cu at (100.7, 127.7)
- added C17: 100nF 100V, Capacitor_SMD:C_0805_2012Metric, F.Cu at (96.3, 127.7)
- added C18: 220nF 16V, Capacitor_SMD:C_0603_1608Metric, F.Cu at (134.6, 130.4)
- added C19: 100nF 100V, Capacitor_SMD:C_0805_2012Metric, F.Cu at (130.4, 127.7)
- added C20: 100nF 100V, Capacitor_SMD:C_0805_2012Metric, F.Cu at (126.0, 127.7)
- added C21: 220nF 16V, Capacitor_SMD:C_0603_1608Metric, F.Cu at (189.2, 81.7)
- added C22: 100nF 100V, Capacitor_SMD:C_0805_2012Metric, F.Cu at (185.0, 78.9)
- added C23: 100nF 100V, Capacitor_SMD:C_0805_2012Metric, F.Cu at (180.6, 78.9)
- added C8: 10uF 50V, Capacitor_SMD:C_0805_2012Metric, F.Cu at (96.3, 113.0)
- added C9: 4.7uF 16V, Capacitor_SMD:C_0805_2012Metric, F.Cu at (105.2, 113.0)
- added D2: LED, LED_SMD:LED_0603_1608Metric, F.Cu at (90.8, 38.7)
- added H1: Solder_Pad, TestPoint:TestPoint_Plated_Hole_D3.0mm, F.Cu at (122.0, 105.6)
- added H2: Solder_Pad, TestPoint:TestPoint_Plated_Hole_D3.0mm, F.Cu at (153.9, 78.5)
- added H3: Solder_Pad, TestPoint:TestPoint_Plated_Hole_D3.0mm, F.Cu at (126.3, 99.3)
- added H4: Solder_Pad, TestPoint:TestPoint_Plated_Hole_D3.0mm, F.Cu at (136.7, 89.1)
- added H5: Solder_Pad, TestPoint:TestPoint_Plated_Hole_D3.0mm, F.Cu at (153.9, 72.4)
- added H6: Solder_Pad, TestPoint:TestPoint_Plated_Hole_D3.0mm, F.Cu at (160.0, 72.4)
- added H7: Solder_Pad, TestPoint:TestPoint_Plated_Hole_D3.0mm, F.Cu at (145.5, 78.8)
- added J2: Conn_01x05_Male, Connector_PinHeader_1.27mm:PinHeader_1x05_P1.27mm_Vertical, F.Cu at (121.2, 93.4)
- added J3: Conn_01x02_Male, Connector_PinHeader_1.27mm:PinHeader_1x02_P1.27mm_Vertical, F.Cu at (69.6, 39.6)
- added J4: Conn_01x04_Male, Connector_PinHeader_1.27mm:PinHeader_2x02_P1.27mm_Vertical, F.Cu at (118.2, 112.0)
- added Q7: 80V 80A, Package_TO_SOT_SMD:TO-252-3_TabPin2, F.Cu at (196.6, 73.4)
- added Q8: 80V 80A, Package_TO_SOT_SMD:TO-252-3_TabPin2, F.Cu at (184.4, 73.4)
- added R12: 40.2k, Resistor_SMD:R_0603_1608Metric, F.Cu at (66.9, 49.3)
- added R13: 100k, Resistor_SMD:R_0603_1608Metric, F.Cu at (153.9, 89.5)
- added R14: 6.2k, Resistor_SMD:R_0603_1608Metric, F.Cu at (165.0, 74.0)
- added R15: 220, Resistor_SMD:R_0603_1608Metric, F.Cu at (163.9, 79.2)
- added R16: 210k, Resistor_SMD:R_0603_1608Metric, F.Cu at (63.2, 50.2)
- added R17: 10, Resistor_SMD:R_0805_2012Metric, F.Cu at (144.3, 83.3)
- added R18: 1k, Resistor_SMD:R_0603_1608Metric, F.Cu at (123.6, 112.5)
- added R20: 5m, gmr320:GMR320, F.Cu at (137.9, 83.3)
- added R21: 180k, Resistor_SMD:R_0603_1608Metric, F.Cu at (169.0, 74.0)
- added R22: 180k, Resistor_SMD:R_0603_1608Metric, F.Cu at (127.6, 112.5)
- added R23: 10, Resistor_SMD:R_0805_2012Metric, F.Cu at (100.7, 130.7)
- added R24: 10, Resistor_SMD:R_0805_2012Metric, F.Cu at (96.2, 130.7)
- added R25: 100k, Resistor_SMD:R_0603_1608Metric, F.Cu at (108.9, 129.9)
- added R26: 100k, Resistor_SMD:R_0603_1608Metric, F.Cu at (108.9, 127.4)
- added R27: 10, Resistor_SMD:R_0805_2012Metric, F.Cu at (130.4, 130.7)
- added R28: 10, Resistor_SMD:R_0805_2012Metric, F.Cu at (125.9, 130.7)
- added R29: 100k, Resistor_SMD:R_0603_1608Metric, F.Cu at (138.6, 129.9)
- added R30: 100k, Resistor_SMD:R_0603_1608Metric, F.Cu at (138.6, 127.4)
- added R31: 10, Resistor_SMD:R_0805_2012Metric, F.Cu at (185.0, 81.9)
- added R32: 10, Resistor_SMD:R_0805_2012Metric, F.Cu at (180.6, 81.9)
- added R33: 100k, Resistor_SMD:R_0603_1608Metric, F.Cu at (193.2, 81.2)
- added R34: 100k, Resistor_SMD:R_0603_1608Metric, F.Cu at (193.2, 78.7)
- added RV1: 25k, Potentiometer_THT:Potentiometer_Bourns_3386F_Vertical, F.Cu at (134.3, 77.5)
- added RV2: 25k, Potentiometer_THT:Potentiometer_Bourns_3386F_Vertical, F.Cu at (125.5, 88.7)
- added RV3: 25k, Potentiometer_THT:Potentiometer_Bourns_3386F_Vertical, F.Cu at (111.0, 99.6)
- added TP1: TestPoint, Connector_PinHeader_1.27mm:PinHeader_1x01_P1.27mm_Vertical, F.Cu at (136.4, 102.9)
- added TP10: TestPoint, Connector_PinHeader_1.27mm:PinHeader_1x01_P1.27mm_Vertical, F.Cu at (152.8, 86.5)
- added TP2: TestPoint, TestPoint:TestPoint_Loop_D2.50mm_Drill1.0mm, F.Cu at (135.8, 98.9)
- added TP3: TestPoint, Connector_PinHeader_1.27mm:PinHeader_1x01_P1.27mm_Vertical, F.Cu at (165.1, 71.0)
- added TP4: TestPoint, Connector_PinHeader_1.27mm:PinHeader_1x01_P1.27mm_Vertical, F.Cu at (152.8, 83.2)
- added TP5: TestPoint, Connector_PinHeader_1.27mm:PinHeader_1x01_P1.27mm_Vertical, F.Cu at (89.7, 49.0)
- added TP6: TestPoint, Connector_PinHeader_1.27mm:PinHeader_1x01_P1.27mm_Vertical, F.Cu at (132.2, 102.9)
- added TP7: TestPoint, Connector_PinHeader_1.27mm:PinHeader_1x01_P1.27mm_Vertical, F.Cu at (159.0, 81.5)
- added TP8: TestPoint, Connector_PinHeader_1.27mm:PinHeader_1x01_P1.27mm_Vertical, F.Cu at (132.2, 106.2)
- added TP9: TestPoint, Connector_PinHeader_1.27mm:PinHeader_1x01_P1.27mm_Vertical, F.Cu at (148.6, 83.5)
- added U3: MP2565DN-LF-Z, Package_SO:SOIC-8-1EP_3.9x4.9mm_P1.27mm_EP2.41x3.3mm_ThermalVias, F.Cu at (70.7, 53.5)
- added U4: TL431DBZ, Package_TO_SOT_SMD:SOT-23, F.Cu at (127.4, 109.0)
- added U5: TL431DBZ, Package_TO_SOT_SMD:SOT-23, F.Cu at (159.4, 77.7)
- added U6: A4915_LP, Package_SO:HTSSOP-28-1EP_4.4x9.7mm_P0.65mm_EP2.85x5.4mm_ThermalVias, F.Cu at (127.0, 75.0)
- added U7: INA310B1 100V/V, Package_SO:VSSOP-8_3.0x3.0mm_P0.65mm, F.Cu at (112.1, 112.6)
- added U8: INA310B1 20V/V, Package_SO:VSSOP-8_3.0x3.0mm_P0.65mm, F.Cu at (127.3, 94.0)
- C1: value 220nF 16V -> 10uF 50V; footprint Capacitor_SMD:C_0603_1608Metric -> Capacitor_SMD:C_0805_2012Metric
- C2: value 220nF 16V -> 100nF 6.3V
- C4: value 22uF 6.3V -> 4.7uF 6.3V
- C5: value 10uF 50V -> 0.47uF 16V; footprint Capacitor_SMD:C_0805_2012Metric -> Capacitor_SMD:C_0603_1608Metric
- C6: value 4.7uF 16V -> 0.47uF 16V; footprint Capacitor_SMD:C_0805_2012Metric -> Capacitor_SMD:C_0603_1608Metric
- C7: value 220nF 16V -> 22uF 6.3V
- J1: value Conn_01x02_Male -> Conn_01x03_Male; footprint Connector_PinHeader_1.27mm:PinHeader_1x02_P1.27mm_Vertical -> Connector_PinHeader_1.27mm:PinHeader_1x03_P1.27mm_Vertical
- Q1: value 80V 80A -> BSS84; footprint Package_TO_SOT_SMD:TO-252-3_TabPin2 -> Package_TO_SOT_SMD:SOT-23
- R1, R11, R9: value 10 -> 1k; footprint Resistor_SMD:R_0805_2012Metric -> Resistor_SMD:R_0603_1608Metric
- R10: value 10 -> 100k; footprint Resistor_SMD:R_0805_2012Metric -> Resistor_SMD:R_0603_1608Metric
- R19: value 10 -> 220; footprint Resistor_SMD:R_0805_2012Metric -> Resistor_SMD:R_0603_1608Metric
- R3: value 10 -> 17.4k; footprint Resistor_SMD:R_0805_2012Metric -> Resistor_SMD:R_0603_1608Metric
- R4: value 17.4k -> 1k
- R5: value 100k -> 200k
- R6: value 40.2k -> 1k
- R7: value 210k -> 64k
- R8: value 200k -> 10k
- U1: value A4915_LP -> MCP6L01Rx-xOT; footprint Package_SO:HTSSOP-28-1EP_4.4x9.7mm_P0.65mm_EP2.85x5.4mm_ThermalVias -> Package_TO_SOT_SMD:SOT-23-5
- U2: value MP2565DN-LF-Z -> MCP6L01Rx-xOT; footprint Package_SO:SOIC-8-1EP_3.9x4.9mm_P1.27mm_EP2.41x3.3mm_ThermalVias -> Package_TO_SOT_SMD:SOT-23-5
- moved R3 125.6 mm to (71.4, 47.3), turned to 90 degrees
- moved R10 123.0 mm to (66.9, 44.8), turned to -90 degrees
- moved C2 115.6 mm to (76.1, 54.0), turned to -90 degrees
- moved C1 112.6 mm to (72.3, 59.7)
- moved C3 109.5 mm to (68.6, 47.4), turned to 90 degrees
- moved R2 109.1 mm to (73.0, 47.2), turned to -90 degrees
- moved R5 104.5 mm to (68.3, 59.6), turned to 180 degrees
- moved D1 88.5 mm to (82.0, 55.9), turned to -90 degrees
- moved R19 86.4 mm to (90.8, 42.3), turned to 90 degrees
- moved Q4 83.1 mm to (100.1, 122.1)
- moved Q5 79.6 mm to (142.0, 122.1)
- moved Q6 79.6 mm to (129.8, 122.1)
- moved L1 79.3 mm to (80.8, 43.7)
- moved C7 76.3 mm to (87.1, 59.3), turned to 180 degrees
- moved Q3 57.6 mm to (112.3, 122.1)
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Connections:
- C1 pad 1: /power stage1/M -> /V_BUS
- C1 pad 2: /power stage1/C -> GND
- C2 pad 1: /power stage2/M -> /SW
- C2 pad 2: /power stage2/C -> Net-(C2-Pad2)
- C4 pad 1: /5V -> Net-(C4-Pad1)
- C5 pad 1: /VBAT -> Net-(C5-Pad1)
- C5 pad 2: GND -> Net-(C5-Pad2)
- C6 pad 1: Net-(U1-Pad14) -> GND
- C6 pad 2: GND -> /5V
- C7 pad 1: /power stage/M -> /5V
- C7 pad 2: /power stage/C -> GND
- D1 pad 1: Net-(D1-Pad1) -> /SW
- J1 pad 1: Net-(U2-Pad2) -> /5V
- J1 pad 2: GND -> Net-(J1-Pad2)
- L1 pad 1: Net-(D1-Pad1) -> /SW
- Q1 pad 2: /power stage1/PH -> /VREG
- Q1 pad 3: /power stage1/M -> Net-(Q1-Pad3)
- Q2 pad 2: /power stage/M -> Net-(H2-Pad1)
- Q2 pad 3: /power stage/PL -> GND
- Q3 pad 2: /power stage/PH -> /V_BUS
- Q3 pad 3: /power stage/M -> /FET stage C/M
- Q4 pad 2: /power stage1/M -> /FET stage C/M
- Q4 pad 3: /power stage1/PL -> /SHUNT_H
- Q5 pad 2: /power stage2/PH -> /V_BUS
- Q5 pad 3: /power stage2/M -> /FET stage A/M
- Q6 pad 2: /power stage2/M -> /FET stage A/M
- Q6 pad 3: /power stage2/PL -> /SHUNT_H
- R1 pad 1: /power stage1/GH -> /5V
- R1 pad 2: Net-(Q1-Pad1) -> /ENABLE
- R10 pad 1: /power stage1/GL -> Net-(C3-Pad2)
- R10 pad 2: Net-(Q4-Pad1) -> GND
- R11 pad 1: /power stage2/GL -> Net-(C4-Pad1)
- R11 pad 2: Net-(Q6-Pad1) -> /CHG_LIM_OD
- R19 pad 1: /power stage/GH -> /5V
- R19 pad 2: Net-(Q3-Pad1) -> Net-(D2-Pad2)
- R2 pad 1: /VBAT -> /V_BUS
- R2 pad 2: Net-(U2-Pad2) -> Net-(J3-Pad1)
- R3 pad 1: /power stage2/GH -> Net-(J3-Pad1)
- R3 pad 2: Net-(Q5-Pad1) -> GND
- R4 pad 1: Net-(U2-Pad2) -> /BRAKEn
- R4 pad 2: GND -> /5V
- R5 pad 1: Net-(C3-Pad2) -> Net-(R5-Pad1)
- R6 pad 1: Net-(R6-Pad1) -> /DIR
- R6 pad 2: GND -> /5V
- R7 pad 1: Net-(R6-Pad1) -> GND
- R7 pad 2: /5V -> /TDEAD
- R8 pad 1: Net-(U2-Pad6) -> /5V
- R8 pad 2: GND -> /FAULT
- R9 pad 1: /power stage/GL -> /CHG_LIM_OD
- R9 pad 2: Net-(Q2-Pad1) -> Net-(R9-Pad2)
- U1 pad 1: unconnected-(U1-Pad1) -> Net-(U1-Pad1)
- U1 pad 2: /power stage/GL -> /5V
- U1 pad 3: /power stage/GH -> Net-(J1-Pad2)
- U1 pad 4: /power stage/M -> Net-(U1-Pad1)
- U1 pad 5: /power stage/C -> GND
- U2 pad 1: Net-(D1-Pad1) -> Net-(R9-Pad2)
- U2 pad 2: Net-(U2-Pad2) -> /5V
- U2 pad 3: Net-(C3-Pad1) -> Net-(RV1-Pad2)
- U2 pad 4: Net-(R6-Pad1) -> Net-(R9-Pad2)
Routing:
- net /5V: track 0.00 -> 40.6 mm, vias 0 -> 1
- net /V_BUS: track 0.00 -> 24.1 mm, vias 0 -> 2
- net GND: track 0.00 -> 15.3 mm, vias 0 -> 17
- net Net-(J3-Pad1): track 0.00 -> 13.8 mm
- net Net-(R12-Pad1): track 0.00 -> 5.11 mm
- net Net-(R5-Pad1): track 0.00 -> 4.02 mm
- net Net-(C2-Pad2): track 0.00 -> 3.92 mm
- net Net-(C3-Pad1): track 0.00 -> 3.48 mm
- net Net-(C3-Pad2): track 0.00 -> 3.27 mm
- net Net-(D2-Pad2): track 0.00 -> 1.94 mm
- added copper zone on F.Cu, net /5V
- added copper zone on F.Cu, net /SW
- added copper zone on F.Cu, net GND
- added copper zone on In2.Cu, net GND
Other:
- copper layers 2 -> 4
