File: SimpleSensoredBldcController.kicad_sch (KiCad schematic)
At the start: 39 parts, among them J1 Conn_01x02_Male, U1 A4915_LP, U2 MP2565DN-LF-Z

Commit message: Lots of progress.
Parts:
- removed R? (x2): 20k, Resistor_SMD:R_0603_1608Metric, symbol Device:R_US
- removed R? (x2): 1k, Resistor_SMD:R_0603_1608Metric, symbol Device:R_US
- removed U? (x3): LMV358, symbol Amplifier_Operational:LMV358
- removed U? (x3): LM319, symbol Comparator:LM319
- added C10: 0.47uF 16V, Capacitor_SMD:C_0603_1608Metric, symbol Device:C
- added C11: 10uF 50V, Capacitor_SMD:C_0805_2012Metric, symbol Device:C
- added C12, C13, C14: 470uF 63V, Capacitor_THT:C_Radial_D12.5mm_H25.0mm_P5.00mm, symbol Device:C
- added C21, C22, C23: 100nF 6.3V, Capacitor_SMD:C_0603_1608Metric, symbol Device:C
- added D2: LED, LED_SMD:LED_0603_1608Metric, symbol Device:LED
- added H1, H2, H3, H4, H5, H6, H7: Solder_Pad, TestPoint:TestPoint_Plated_Hole_D3.0mm, symbol Mechanical:MountingHole_Pad
- added J2: Conn_01x03_Male, Connector_PinHeader_1.27mm:PinHeader_1x03_P1.27mm_Vertical, symbol Connector:Conn_01x03_Male
- added Q7: BSS84, Package_TO_SOT_SMD:SOT-23, symbol Transistor_FET:BSS84
- added Q8: 80V 80A, Package_TO_SOT_SMD:TO-252-3_TabPin2, symbol Device:Q_NMOS_GDS
- added R22, R24: 220, Resistor_SMD:R_0603_1608Metric, symbol Device:R_US
- added R25: 10, Resistor_SMD:R_0805_2012Metric, symbol Device:R_US
- added R26: 1k, Resistor_SMD:R_0603_1608Metric, symbol Device:R_US
- added R27, R34: 180k, Resistor_SMD:R_0603_1608Metric, symbol Device:R_US
- added RV1, RV2: 25k, Potentiometer_THT:Potentiometer_Bourns_3386F_Vertical, symbol Device:R_Potentiometer_Trim_US
- added TP2, TP4, TP6: TestPoint, TestPoint:TestPoint_Loop_D2.50mm_Drill1.0mm, symbol Connector:TestPoint
- added U3: MCP6L01Rx-xOT, Package_TO_SOT_SMD:SOT-23-5, symbol Amplifier_Operational:MCP6L01Rx-xOT
- added U4, U5: TL431DBZ, Package_TO_SOT_SMD:SOT-23, symbol Reference_Voltage:TL431DBZ
- added U6: INA310B1 100V/V, Package_SO:VSSOP-8_3.0x3.0mm_P0.65mm, symbol INA310X:INA310x
- added U7: INA310B1 20V/V, Package_SO:VSSOP-8_3.0x3.0mm_P0.65mm, symbol INA310X:INA310x
- R21: renamed from R?; value 10k -> 6.2k; MPN RC0603FR-0710KL -> RC0603FR-076K2L; VPN1 311-10.0KHRCT-ND -> 311-6.20KHRCT-ND
- gave numbers to parts that had none: 13
Connections:
- net VBAT is gone; now on net V_BUS: C5.1, R2.1, U2.7 (VIN)
- net 5V: now also C10.2, J2.1 (Pin_1), R22.1, TP4.1, U3.2 (V+)
- net BRAKEn: now also J3.4 (Pin_4), R15.1
- net CHG_LIM_OD: now also U6.6 (CMP_OUT), U7.6 (CMP_OUT)
- net ENABLE: now also U4.1 (K)
- net GND: now also C10.1, C11.2, C12.2, C13.2, C14.2, C22.2, C23.2, D2.1 (K), H5.1, J2.3 (Pin_3), Q8.3 (S), R26.2, R27.1, R34.1, U3.5 (V-), U4.3 (A), U5.3 (A), U6.4 (GND), U6.5 (RESET), U6.8 (IN+), U7.4 (GND), U7.5 (RESET), U7.7 (IN-)
- net HC: now also J4.4 (Pin_4)
- net V_BUS: now also C11.1, C12.1, C13.1, C14.1, H4.1, H6.1
- net power stage/M: now also H3.1
- net power stage1/M: now also H1.1
- net power stage2/M: now also H2.1
- net at R20.2, R21.1: now also U5.2 (REF)
- net at D1.1 (K), L1.1, U2.1 (SW): now also C21.1
- net SHUNT_H: now reaches R23.2, U1.1 (LSS)
- net SHUNT_H: now also U6.7 (IN-), U7.8 (IN+)
- net VREG: now reaches C6.1, U1.14 (VREG)
- net VREG: now also Q7.2 (S), R24.1, TP6.1
- net at U2.8 (BST): now also C21.2
- net SPD_IN: no longer names the net of R17.2
- net SPD_IN: now also TP2.1, U3.1, U3.4 (-)
- new net: Q7.1 (G), R24.2, U5.1 (K)
- new net: C23.1, U7.1 (V_S)
- new net: RV2.3, U7.2 (OUT)
- new net: RV2.2, U7.3 (CMP_IN)
- new net: J2.2 (Pin_2), U3.3 (+)
- new net: Q8.1 (G), R25.1, R26.1
- new net: Q7.3 (D), R25.2
- new net: R34.2, RV2.1
- new net: H7.1, Q8.2 (D)
- new net: D2.2 (A), R22.2
- new net: C22.1, U6.1 (V_S)
- new net: RV1.3, U6.2 (OUT)
- new net: RV1.2, U6.3 (CMP_IN)
- new net: R27.2, RV1.1
Other:
- note added: "0.005V/A"
- note added: "0.5V/A"
- note added: "43V Voltage limit"
- note added: "Speed control potentiometer"
- note added: "This divider maps the max output of 5V to the trip voltage of 0.6V."
- note added: "To be placed close to the three power stages"
- note added: "Todo * Make testpoint footprints pin headers * Hook up power stages to power"
- note added: "Trips between 1.2A and 10A"
- note added: "Trips between 6A and 50A"
- note added: "charge current limiter"
- note added: "discharge current limiter"
- note removed: "2.38A charge current limit"
- note removed: "45V Voltage limit"
- note removed: "TODO: * Potentiometer connector * 5V power LED * ELKOs * Gate/Source resistors * Battery and motor pads"
- moved on the sheet: R13, R14

Commit message: Started routing.
Parts:
- added RV1: 25k, Potentiometer_THT:Potentiometer_Bourns_3386F_Vertical, symbol Device:R_Potentiometer_Trim_US
- added TP1, TP10, TP3, TP5, TP6, TP8, TP9: TestPoint, Connector_PinHeader_1.27mm:PinHeader_1x01_P1.27mm_Vertical, symbol Connector:TestPoint
- added U2: MCP6L01Rx-xOT, Package_TO_SOT_SMD:SOT-23-5, symbol Amplifier_Operational:MCP6L01Rx-xOT
- TP4: footprint TestPoint:TestPoint_Loop_D2.50mm_Drill1.0mm -> Connector_PinHeader_1.27mm:PinHeader_1x01_P1.27mm_Vertical
- TP7: renamed from TP6; footprint TestPoint:TestPoint_Loop_D2.50mm_Drill1.0mm -> Connector_PinHeader_1.27mm:PinHeader_1x01_P1.27mm_Vertical
- renumbered C5 to C1, C12 to C10, C22 to C11, C13 to C12, C23 to C13, C21 to C2, C8 to C4, C9 to C5, C10 to C6, C4 to C7, C11 to C8, C6 to C9, H6 to H1, H7 to H2, H1 to H3, H2 to H4, H3 to H5, H4 to H6, H5 to H7, J2 to J1, J4 to J2, J1 to J3, J3 to J4, Q7 to Q1, Q8 to Q2, R13 to R1, R5 to R10, R18 to R11, R6 to R12, R20 to R13, R21 to R14, R24 to R15, R7 to R16, R25 to R17, R26 to R18, R22 to R19, R23 to R20, R27 to R21, R34 to R22, R4 to R3, R15 to R4, R8 to R5, R16 to R6, R12 to R7, R14 to R8, R17 to R9, RV1 to RV2, RV2 to RV3, U3 to U1, U2 to U3, U1 to U6, U6 to U7, U7 to U8
Connections:
- net 5V: now also TP5.1, U2.2 (V+); no longer TP4.1
- net GND: now also RV1.3, U2.5 (V-)
- net V_BUS: now also TP8.1
- net at R9.2, TP2.1: now also TP3.1, U2.1, U2.4 (-); no longer U1.1, U1.4 (-)
- net at R13.2, R14.1, U5.2 (REF): now also TP4.1
- net SW: now reaches C2.1, D1.1 (K), L1.1, U3.1 (SW)
- net at RV3.2, U8.3 (CMP_IN): now also TP10.1
- net at Q2.1 (G), R17.1, R18.1: now also TP6.1
- net at RV2.2, U7.3 (CMP_IN): now also TP9.1
- net SHUNT_H renamed LSS
- new net: U1.1, U1.4 (-)
- new net: RV1.1, TP1.1
- new net: RV1.2, U2.3 (+)
Other:
- sheet power stage renamed FET stage C
- sheet power stage1 renamed FET stage A
- sheet power stage2 renamed FET stage B
- note added: "Input range selection potentiometer"
- note added: "To speed input potentiometer"
- note removed: "Speed control potentiometer"
- note removed: "Todo * Make testpoint footprints pin headers * Hook up power stages to power"
- moved on the sheet: J1, J2, R7, R8, U1
